File: products/WM1-watermaster/hardware/ValveNode/ValveNode.kicad_sch (KiCad schematic)
At the start: 37 parts, among them J1 Conn_IN, J2 Conn_Coaxial_Small, J3 PWR_CONN, J4 Relay_CONN, K1 Cube_Relay, U1 ULN2003, U13 AMS1117-5.0, U5 ESP32 30 Pin CP2102 Developme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, U7 ISC-SX1262-B, U8 AP2112K-3.3

Commit message: Update Nursary_OneCH hardware
Parts:
- removed C3, C8: 100pF, Capacitor_SMD:C_0805_2012Metric, symbol Device:C
- removed D4: LED_GREEN_IN1, LED_SMD:LED_0603_1608Metric, symbol Device:LED
- removed D5: LED_RED_IN4, LED_SMD:LED_0603_1608Metric, symbol Device:LED
- removed D6, D7: PESD3V3U1UL, Diode_SMD:D_SOD-882, symbol Diode:PESD3V3U1UL
- removed J1: Conn_IN, Connector_Phoenix_MSTB:PhoenixContact_MSTBA_2,5_3-G-5,08_1x03_P5.08mm_Horizontal, symbol Connector:Conn_01x03_Pin
- removed J4: Relay_CONN, PhoenixContact_MSTBA_2,5_2-G-5,08_1x02_P5.08mm_Horizontal, symbol Connector:Conn_01x02_Pin
- removed K1: Cube_Relay, Relay_THT:Relay_SPDT_SANYOU_SRD_Series_Form_C, symbol Relay:SANYOU_SRD_Form_C
- removed R11, R6, R8, R9: 470E, Resistor_SMD:R_0805_2012Metric, symbol Device:R
- removed R12, R7: 10K, Resistor_SMD:R_0805_2012Metric, symbol Device:R
- removed U1: ULN2003, Package_SO:SOIC-16W_5.3x10.2mm_P1.27mm, symbol Transistor_Array:ULN2003
- added C1, C9: 100nF, Capacitor_SMD:C_0805_2012Metric, symbol Device:C
- added C11, C15, C2: 1000mfd,25V, Capacitor_THT:CP_Radial_D10.0mm_P2.50mm_P5.00mm, symbol Device:C_US
- added J5: Conn_01x05_Pin, Connector_Phoenix_MSTB:PhoenixContact_MSTBA_2,5_5-G-5,08_1x05_P5.08mm_Horizontal, symbol Connector:Conn_01x05_Pin
- added R10, R15, R3, R4: 22K, Resistor_SMD:R_0805_2012Metric, symbol Device:R
- added U10, U4, U6, U9: DRV8871DDA, Package_SO:Texas_HTSOP-8-1EP_3.9x4.9mm_P1.27mm_EP2.95x4.9mm_Mask2.4x3.1mm_ThermalVias, symbol Driver_Motor:DRV8871DDA
- added U11, U2: 74HC595, Package_SO:SOIC-16_3.9x9.9mm_P1.27mm, symbol 74xx:74HC595
- D3: value LED_YELLOW_PUMP -> LED_Valve_Yellow
Connections:
- net +3.3V: now also C1.1, C9.1, U11.10 (~{SRCLR}), U11.16 (VCC), U2.10 (~{SRCLR}), U2.16 (VCC)
- net +8V: now also C11.1, C15.1, C2.1, U10.5 (VM), U4.5 (VM), U6.5 (VM), U9.5 (VM)
- net GND: now also C1.2, C11.2, C15.2, C2.2, C9.2, R10.2, R15.2, R3.2, R4.2, U10.1 (GND), U10.7 (GND), U10.9 (GND), U11.13 (~{OE}), U11.8 (GND), U2.13 (~{OE}), U2.8 (GND), U4.1 (GND), U4.7 (GND), U4.9 (GND), U6.1 (GND), U6.7 (GND), U6.9 (GND), U9.1 (GND), U9.7 (GND), U9.9 (GND)
- net Valve_DATA: now reaches U5.7 (Tx2/D17)
- net Valve_DATA: now also U2.14 (SER)
- net IN1_LED_MCU: no longer names the net of U5.22 (D33)
- net IN1_MCU: no longer names the net of U5.17 (VP(36)/Input_only)
- net IN4_LED_MCU renamed Valve_LATCH
- net Valve_LATCH: now also U11.12 (RCLK), U2.12 (RCLK)
- net IN4_MCU: no longer names the net of U5.20 (D35/Input_only)
- net Pump_ON_Yellow_LED renamed Any_Valve_Activity_LED
- net Any_Valve_Activity_LED: now also U11.5 (QF); no longer U5.6 (Rx2/D16)
- net RELAY1_MCU: no longer names the net of U5.21 (D32)
- new net: R15.1, U6.4 (ILIM)
- new net: R4.1, U9.4 (ILIM)
- new net: R10.1, U10.4 (ILIM)
- new net: R3.1, U4.4 (ILIM)
- new net NoPWR_LED: U11.4 (QE)
- new net RLY_DATA_EXT: U11.9 (QH')
- new net SER1_OUT: U11.14 (SER), U2.9 (QH')
- new net V1_IN1: U2.15 (QA), U4.3 (IN1)
- new net V1_IN2: U2.1 (QB), U4.2 (IN2)
- new net V1_LED: U11.15 (QA)
- new net V1_OUT: J5.4 (Pin_4), U4.8 (OUT2)
- new net V2_IN1: U2.2 (QC), U6.3 (IN1)
- new net V2_IN2: U2.3 (QD), U6.2 (IN2)
- new net V2_LED: U11.1 (QB)
- new net V2_OUT: J5.3 (Pin_3), U6.8 (OUT2)
- new net V3_IN1: U2.4 (QE), U9.3 (IN1)
- new net V3_IN2: U2.5 (QF), U9.2 (IN2)
- new net V3_LED: U11.2 (QC)
- new net V3_OUT: J5.2 (Pin_2), U9.8 (OUT2)
- new net V4_IN1: U10.3 (IN1), U2.6 (QG)
- new net V4_IN2: U10.2 (IN2), U2.7 (QH)
- new net V4_LED: U11.3 (QD)
- new net V4_OUT: J5.1 (Pin_1), U10.8 (OUT2)
- new net V_Com_OUT: J5.5 (Pin_5), U10.6 (OUT1), U4.6 (OUT1), U6.6 (OUT1), U9.6 (OUT1)
- new net Valve_CLK: U11.11 (SRCLK), U2.11 (SRCLK), U5.6 (Rx2/D16)
- no-connect marks 15 -> 20
Other:
- note added: "Latch Valve control"
- note removed: "Close to MCU"
- note removed: "Close to connector"
- note removed: "No Power INPUT"
- note removed: "RL1"
- note removed: "Relay OUTPUT"
- note removed: "Water Flow INPUT"
- moved on the sheet: C10, C12, C13, C4, C5, C6, C7, D1, D2, H1, J2, J3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
