File: products/WM1-watermaster/hardware/ValveNode/ValveNode.kicad_sch (KiCad schematic)
At the start: 37 parts, among them J2 Conn_Coaxial_Small, J3 PWR_CONN, J5 Conn_01x05_Pin, U10 DRV8871DDA, U11 74HC595, U13 AMS1117-5.0, U2 74HC595, U4 DRV8871DDA, U5 ESP32 30 Pin CP2102 Developme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, U6 DRV8871DDA, U7 ISC-SX1262-B, U8 AP2112K-3.3, U9 DRV8871DDA

Commit message: Update Nursary_OneCH hardware
Parts:
- added C19: 100nF, Capacitor_SMD:C_0805_2012Metric, symbol Device:C
- added D16: PESD3V3U1UL, Diode_SMD:D_SOD-882, symbol Diode:PESD3V3U1UL
- added R18: 56.2K, Resistor_SMD:R_0805_2012Metric, symbol Device:R
- added R32: 10K, Resistor_SMD:R_0805_2012Metric, symbol Device:R
- added R33: 470E, Resistor_SMD:R_0805_2012Metric, symbol Device:R
Connections:
- net +8V: now also R18.1
- net GND: now also C19.2, D16.2 (A), R32.2
- net Batt_Mon: now reaches U5.20 (D35/Input_only)
- net Batt_Mon: now also C19.1, R33.1
- new net: D16.1 (K), R18.2, R32.1, R33.2
- no-connect marks 20 -> 19
Other:
- note added: "Close to MCU"
- note added: "Close to connector"
