File: products/WM1-watermaster/hardware/ValveNode/ValveNode.kicad_pcb (KiCad board)
At the start: 2 copper layers, 83 x 72 mm, 45 parts, among them J1 Conn_IN, J2 Conn_Coaxial_Small, J3 PWR_CONN, J4 Relay_CONN, K1 Cube_Relay, U1 ULN2003, U13 AMS1117-5.0, U5 ESP32 30 Pin CP2102 Developme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, U7 ISC-SX1262-B, U8 AP2112K-3.3

Commit message: Update Nursary_OneCH hardware
Parts:
- removed C3, C8: 100pF, Capacitor_SMD:C_0805_2012Metric
- removed D4: LED_GREEN_IN1, LED_SMD:LED_0603_1608Metric
- removed D5: LED_RED_IN4, LED_SMD:LED_0603_1608Metric
- removed D6, D7: PESD3V3U1UL, Diode_SMD:D_SOD-882
- removed J1: Conn_IN, Connector_Phoenix_MSTB:PhoenixContact_MSTBA_2,5_3-G-5,08_1x03_P5.08mm_Horizontal
- removed J4: Relay_CONN, Connector_Phoenix_MSTB:PhoenixContact_MSTBA_2,5_2-G-5,08_1x02_P5.08mm_Horizontal
- removed K1: Cube_Relay, Relay_THT:Relay_SPDT_SANYOU_SRD_Series_Form_C
- removed R11, R6, R8, R9: 470E, Resistor_SMD:R_0805_2012Metric
- removed R12, R7: 10K, Resistor_SMD:R_0805_2012Metric
- removed U1: ULN2003, Package_SO:SOIC-16W_5.3x10.2mm_P1.27mm
- added C1: 100nF, Capacitor_SMD:C_0805_2012Metric, B.Cu at (169.6, 54.1)
- added C11: 1000mfd,25V, Capacitor_THT:CP_Radial_D10.0mm_P2.50mm_P5.00mm, F.Cu at (160.2, 67.5)
- added C15: 1000mfd,25V, Capacitor_THT:CP_Radial_D10.0mm_P2.50mm_P5.00mm, F.Cu at (170.1, 70.8)
- added C2: 1000mfd,25V, Capacitor_THT:CP_Radial_D10.0mm_P2.50mm_P5.00mm, F.Cu at (180.1, 67.5)
- added C9: 100nF, Capacitor_SMD:C_0805_2012Metric, B.Cu at (169.6, 57.1)
- added J5: Conn_01x05_Pin, Connector_Phoenix_MSTB:PhoenixContact_MSTBA_2,5_5-G-5,08_1x05_P5.08mm_Horizontal, F.Cu at (163.1, 80.8)
- added R10: 22K, Resistor_SMD:R_0805_2012Metric, B.Cu at (160.3, 67.9)
- added R15: 22K, Resistor_SMD:R_0805_2012Metric, B.Cu at (173.1, 68.4)
- added R3: 22K, Resistor_SMD:R_0805_2012Metric, B.Cu at (179.6, 67.5)
- added R4: 22K, Resistor_SMD:R_0805_2012Metric, B.Cu at (166.8, 68.0)
- added U10: DRV8871DDA, Package_SO:Texas_HTSOP-8-1EP_3.9x4.9mm_P1.27mm_EP2.95x4.9mm_Mask2.4x3.1mm_ThermalVias, B.Cu at (157.6, 73.2)
- added U11: 74HC595, Package_SO:SOIC-16_3.9x9.9mm_P1.27mm, B.Cu at (176.3, 62.1)
- added U2: 74HC595, Package_SO:SOIC-16_3.9x9.9mm_P1.27mm, B.Cu at (165.0, 62.2)
- added U4: DRV8871DDA, Package_SO:Texas_HTSOP-8-1EP_3.9x4.9mm_P1.27mm_EP2.95x4.9mm_Mask2.4x3.1mm_ThermalVias, B.Cu at (176.8, 73.2)
- added U6: DRV8871DDA, Package_SO:Texas_HTSOP-8-1EP_3.9x4.9mm_P1.27mm_EP2.95x4.9mm_Mask2.4x3.1mm_ThermalVias, B.Cu at (170.5, 73.2)
- added U9: DRV8871DDA, Package_SO:Texas_HTSOP-8-1EP_3.9x4.9mm_P1.27mm_EP2.95x4.9mm_Mask2.4x3.1mm_ThermalVias, B.Cu at (164.1, 73.2)
- C7: moved to F.Cu
- D3: value LED_YELLOW_PUMP -> LED_Valve_Yellow
- moved C7 33.1 mm to (219.1, 136.7), turned to 0 degrees
Connections:
- R5 pad 1: /Pump_ON_Yellow_LED -> /Any_Valve_Activity_LED
- U5 pad 17: /IN1_MCU -> unconnected-(U5-VP(36)/Input_only-Pad17)
- U5 pad 20: /IN4_MCU -> unconnected-(U5-D35/Input_only-Pad20)
- U5 pad 21: /RELAY1_MCU -> unconnected-(U5-D32-Pad21)
- U5 pad 22: /IN1_LED_MCU -> unconnected-(U5-D33-Pad22)
- U5 pad 28: /IN4_LED_MCU -> /Valve_LATCH
- U5 pad 6: /Pump_ON_Yellow_LED -> /Valve_CLK
Routing:
- net Net-(D5-A): track 69.3 -> 0.00 mm, vias 5 -> 0
- net /V_Com_OUT: track 0.00 -> 68.7 mm
- net /RELAY1_MCU: track 63.2 -> 0.00 mm, vias 2 -> 0
- net +5V: track 185.6 -> 128.8 mm, vias 22 -> 19
- net Net-(D4-A): track 46.5 -> 0.00 mm, vias 3 -> 0
- net /IN1_CON: track 38.8 -> 0.00 mm
- net /IN4_CON: track 33.1 -> 0.00 mm
- net +3.3V: track 52.3 -> 25.8 mm, vias 2 -> 0
- net /RLY_COMM: track 21.4 -> 0.00 mm
- net +8V: track 46.5 -> 67.4 mm
- net /RL1_CON_1: track 18.4 -> 0.00 mm
- net /V1_IN1: track 0.00 -> 17.4 mm
- net /IN4_MCU: track 13.4 -> 0.00 mm
- net /IN1_MCU: track 13.0 -> 0.00 mm
- net /V4_OUT: track 0.00 -> 11.2 mm
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Other:
- board text removed: "COM"
- board text removed: "IN1"
- board text removed: "IN2"

Commit message: Update Nursary_OneCH hardware
Parts:
- removed the . at (233.8, 113.1)
- removed the ? at (156.8, 58.1)
- removed the ? at (233.8, 58.1)
- removed the ? at (156.8, 113.1)
- added ?: , , F.Cu at (73.5, 49.0)
- added ?: , , F.Cu at (73.5, 133.0)
- added ?: , , F.Cu at (43.5, 49.0)
- added ?: , , F.Cu at (43.5, 133.0)
- added C19: 100nF, Capacitor_SMD:C_0805_2012Metric, F.Cu at (81.1, 142.3)
- added D16: PESD3V3U1UL, Diode_SMD:D_SOD-882, F.Cu at (80.3, 144.9)
- added R18: 56.2K, Resistor_SMD:R_0805_2012Metric, F.Cu at (76.7, 142.2)
- added R32: 10K, Resistor_SMD:R_0805_2012Metric, F.Cu at (76.7, 145.2)
- added R33: 470E, Resistor_SMD:R_0805_2012Metric, F.Cu at (76.7, 148.1)
- moved U5 173.4 mm to (56.0, 96.0)
- moved C2 160.6 mm to (32.6, 131.1)
- moved C10 155.7 mm to (54.5, 55.5)
- moved U8 155.7 mm to (51.4, 55.5)
- moved C12 155.7 mm to (46.1, 55.4)
- moved C13 155.7 mm to (48.2, 55.4)
- moved C5 154.1 mm to (80.3, 109.2)
- moved U13 152.1 mm to (80.7, 117.6)
- moved C15 146.7 mm to (32.1, 120.8)
- moved C4 134.2 mm to (96.2, 124.8)
- moved J3 128.3 mm to (68.9, 118.1)
- moved J5 128.3 mm to (40.3, 118.2)
- moved J2 126.9 mm to (57.5, 47.2)
- moved U7 122.5 mm to (68.9, 61.1)
- moved R15 121.9 mm to (56.3, 103.4)
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Connections:
- U5 pad 20: unconnected-(U5-D35/Input_only-Pad20) -> /Batt_Mon
Routing:
- net +5V: track 128.8 -> 0.00 mm, vias 19 -> 0
- net /RESET: track 82.4 -> 0.00 mm
- net /DIO1: track 81.1 -> 0.00 mm
- net /NSS: track 77.8 -> 0.00 mm, vias 2 -> 0
- net /V_Com_OUT: track 68.7 -> 0.00 mm
- net +8V: track 67.4 -> 0.00 mm
- net /BUSY: track 66.7 -> 0.00 mm, vias 2 -> 0
- net /SCK: track 62.9 -> 0.00 mm, vias 2 -> 0
- net /MISO: track 60.3 -> 0.00 mm, vias 2 -> 0
- net /MOSI: track 51.0 -> 0.00 mm, vias 2 -> 0
- net +3.3V: track 25.8 -> 0.00 mm
- net +3.3VL: track 19.9 -> 0.00 mm
- net /V1_IN1: track 17.4 -> 0.00 mm
- net Net-(D1-A): track 11.9 -> 0.00 mm
- net /V4_OUT: track 11.2 -> 0.00 mm
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- removed copper zone on B.Cu, net GND
- removed copper zone on F.Cu, net GND
Other:
- board size 83 x 72 mm -> 57.1 x 91.8 mm
- board text removed: "+8V"
- board text removed: "1"
- board text removed: "5V"
- board text removed: "PWR"

Commit message: updated Valve Node-V4
Parts:
- removed C9: 100nF, Capacitor_SMD:C_0805_2012Metric
- removed U11: 74HC595, Package_SO:SOIC-16_3.9x9.9mm_P1.27mm
- added D4: LED_V3_Yellow, LED_SMD:LED_0805_2012Metric_Pad1.15x1.40mm_HandSolder, F.Cu at (83.5, 85.1)
- added D5: LED_V4_Yellow, LED_SMD:LED_0805_2012Metric_Pad1.15x1.40mm_HandSolder, F.Cu at (83.6, 94.7)
- added R6: 470E, Resistor_SMD:R_0805_2012Metric, B.Cu at (83.5, 82.9)
- added R7: 470E, Resistor_SMD:R_0805_2012Metric, B.Cu at (83.5, 91.5)
- C19, C7, D16, R18, R32, R33: moved to B.Cu
- D1: value Power_Green_LED -> LED_V1_Yellow; footprint LED_THT:LED_D3.0mm -> LED_SMD:LED_0805_2012Metric_Pad1.15x1.40mm_HandSolder
- D2: footprint LED_THT:LED_D3.0mm -> LED_SMD:LED_0805_2012Metric_Pad1.15x1.40mm_HandSolder
- D3: value LED_Valve_Yellow -> LED_V2_Yellow; footprint LED_THT:LED_D3.0mm -> LED_SMD:LED_0805_2012Metric_Pad1.15x1.40mm_HandSolder
- J3: footprint Connector_Phoenix_MSTB:PhoenixContact_MSTBA_2,5_2-G-5,08_1x02_P5.08mm_Horizontal -> Connector_Phoenix_MSTB:PhoenixContact_MSTBVA_2,5_2-G-5,08_1x02_P5.08mm_Vertical
- J5: footprint Connector_Phoenix_MSTB:PhoenixContact_MSTBA_2,5_5-G-5,08_1x05_P5.08mm_Horizontal -> Connector_Phoenix_MSTB:PhoenixContact_MSTBVA_2,5_5-G-5,08_1x05_P5.08mm_Vertical
- moved R33 90.4 mm to (36.3, 67.3)
- moved C19 84.6 mm to (36.3, 70.5)
- moved C7 80.1 mm to (30.8, 106.7), turned to 90 degrees
- moved C6 68.0 mm to (42.3, 106.7), turned to 90 degrees
- moved D2 67.3 mm to (70.4, 55.5)
- moved C4 61.7 mm to (34.6, 129.5), turned to -90 degrees
- moved R18 59.0 mm to (40.2, 95.8), turned to 90 degrees
- moved R32 58.6 mm to (45.2, 95.8), turned to -90 degrees
- moved D16 58.6 mm to (48.5, 95.8), turned to -90 degrees
- moved D1 55.9 mm to (83.3, 65.3)
- moved R2 49.5 mm to (82.2, 58.8), turned to 180 degrees
- moved R13 46.6 mm to (60.7, 78.4), turned to 180 degrees
- moved C5 46.5 mm to (34.4, 116.9), turned to -90 degrees
- moved R1 46.4 mm to (83.3, 67.8)
- moved U13 45.7 mm to (36.3, 106.7), turned to -90 degrees
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Connections:
- R1 pad 1: +5V -> /V1_LED
- R5 pad 1: /Any_Valve_Activity_LED -> /V2_LED
- U2 pad 9: /SER1_OUT -> unconnected-(U2-QH'-Pad9)
- U5 pad 21: unconnected-(U5-D32-Pad21) -> /V1_LED
- U5 pad 22: unconnected-(U5-D33-Pad22) -> /V2_LED
- U5 pad 5: /LoRa_LED -> /V4_LED
Routing:
- net +8V: track 0.00 -> 301.1 mm, vias 0 -> 52
- net +5V: track 0.00 -> 95.8 mm, vias 0 -> 10
- net GND: track 0.00 -> 82.3 mm, vias 0 -> 122
- net /DIO1: track 0.00 -> 66.0 mm
- net /V_Com_OUT: track 0.00 -> 64.0 mm
- net /V1_LED: track 0.00 -> 61.4 mm, vias 0 -> 2
- net /BUSY: track 0.00 -> 59.1 mm
- net /RESET: track 0.00 -> 58.6 mm
- net /V3_LED: track 0.00 -> 58.2 mm
- net /V2_LED: track 0.00 -> 55.0 mm, vias 0 -> 3
- net +3.3V: track 0.00 -> 54.9 mm, vias 0 -> 5
- net Net-(D16-K): track 0.00 -> 42.7 mm, vias 0 -> 2
- net /Valve_LATCH: track 0.00 -> 42.2 mm
- net /V4_LED: track 0.00 -> 30.9 mm, vias 0 -> 2
- net /LoRa_LED: track 0.00 -> 30.7 mm, vias 0 -> 2
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- added copper zone on B.Cu, net GND
- added copper zone on F.Cu, net GND
Other:
- board text added: "+8V"
- board text added: "1"
- board text added: "3V3"
- board text added: "5V"
- board text added: "B"
- board text added: "COM"
- board text added: "V1"
- board text added: "V2"
- board text added: "V3"
- board text added: "V4"
- board text added: "Valve Node VN4"
- board text added: "Y"
- board text removed: "3.3V"
- board text removed: "PUMP"
- board text removed: "PUMP Node-PN"
- board text removed: "Pump"
- board text removed: "Pump Node PN"
