File: products/FG1-flowguard/hardware/Nursary_OneCH/Nursary_OneCH.kicad_sch (KiCad schematic)
At the start: 37 parts, among them J1 FLOW1_CONN, J2 Relay1_CONN, J3 PWR_CONN, J4 FLOW2_CONN, K1 Cube_Relay, U1 ULN2003, U3 DS1307Z+, U4 DS3231M, U5 ESP32 30 Pin CP2102 Developme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, Y1 Crystal

Commit message: Update Nursary_OneCH hardware
Parts:
- removed C1, C5: 100nF, Capacitor_SMD:C_0805_2012Metric, symbol Device:C
- removed C2: 200pF, Capacitor_SMD:C_0805_2012Metric, symbol Device:C
- removed D2: PESD3V3U1UL, Diode_SMD:D_SOD-882, symbol Diode:PESD3V3U1UL
- removed D3: LED_GREEN_FLOW, LED_SMD:LED_0603_1608Metric, symbol Device:LED
- removed F2: Polyfuse_Small, Inductor_SMD:L_1206_3216Metric, symbol Device:Polyfuse_Small
- removed J3: PWR_CONN, symbol Connector:Conn_01x02_Pin
- removed J4: FLOW2_CONN, Connector_JST:JST_EH_B3B-EH-A_1x03_P2.50mm_Vertical, symbol Connector:Conn_01x03_Pin
- removed R1: 2K2, Resistor_SMD:R_0805_2012Metric, symbol Device:R
- removed R2, R6: 100E, Resistor_SMD:R_0805_2012Metric, symbol Device:R
- removed R4: 10K, Resistor_SMD:R_0805_2012Metric, symbol Device:R
- removed R8: 470E, Resistor_SMD:R_0805_2012Metric, symbol Device:R
- added J4: Conn_01x02_Pin, JST_PH_B2B-PH-K_1x02_P2.00mm_Vertical, symbol Connector:Conn_01x02_Pin
- C2: renamed from C3; value 200pF -> 100pF
- D1, D4: footprint LED_SMD:LED_0603_1608Metric -> LED_0805_2012Metric
- J1: value FLOW1_CONN -> Conn_IN; footprint Connector_JST:JST_EH_B3B-EH-A_1x03_P2.50mm_Vertical -> Connector_Phoenix_MSTB:PhoenixContact_MSTBVA_2,5_3-G-5,08_1x03_P5.08mm_Vertical
- J2: footprint (none) -> Connector_Phoenix_MSTB:PhoenixContact_MSTBVA_2,5_2-G-5,08_1x02_P5.08mm_Vertical
- R1: renamed from R9; value 2K2 -> 470E
- U1: footprint Package_SO:SOIC-16W_5.3x10.2mm_P1.27mm -> Package_SO:SOIC-16_3.9x9.9mm_P1.27mm
- renumbered D5 to D6, R7 to R4
Connections:
- net +5VR is gone; now on net +5V: C4.1, C6.1, K1.5, R5.1, U1.9 (COM)
- net FLOW1_PROT is gone; now on net GND: D1.1 (K)
- net FLOW2_CONN is gone; now on net FLOW1_CON: D6.1 (K), R1.2
- net FLOW2_PROT is gone; now on net FLOW1_MCU: C2.1, R1.1, R4.2
- net +5V: now also J4.2 (Pin_2)
- net +5VP: no longer R3.1
- net GND: now also J4.1 (Pin_1)
- net FLOW1_LED_MCU: now reaches U5.21 (D32)
- net FLOW1_LED_MCU: now also R3.1
- net at U3.1 (X1): now also Y1.2; no longer Y1.1
- net at U3.2 (X2): now also Y1.1; no longer Y1.2
- net FLOW1_CONN renamed FLOW1_CON
- net FLOW2_MCU: no longer names the net of U5.19 (D34/Input_only)
- no-connect marks 3 -> 15
Other:
- note added: "Close to MCU"
- note added: "RTC (any one to use)"
- note removed: "Close to ESP32"
- note removed: "RTC for GW"
- moved on the sheet: C2, D4, D6, F1, J2, K1, R1, R4, R5, U1, U3, U5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

Commit message: Update Nursary_OneCH hardware
Parts:
- added TP1: TestPoint, TestPoint:TestPoint_Keystone_5019_Miniature, symbol Connector:TestPoint
Connections:
- net GND: now also TP1.1
- no-connect marks 15 -> 36
Changed lines of the file:
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@@
 	)
 	(junction
+		(at 334.01 233.68)
+		(diameter 0)
+		(color 0 0 0 0)
+	)
+	(junction
 		(at 289.56 118.11)
 		(diameter 0)
@@
 	)
 	(no_connect
+		(at 370.84 125.73)
+	)
+	(no_connect
+		(at 314.96 80.01)
+	)
+	(no_connect
+		(at 314.96 106.68)
+	)
+	(no_connect
 		(at 180.34 190.5)
 	)
 	(no_connect
+		(at 314.96 110.49)
+	)
+	(no_connect
+		(at 370.84 114.3)
+	)
+	(no_connect
+		(at 370.84 118.11)
+	)
+	(no_connect
+		(at 314.96 118.11)
+	)
+	(no_connect
+		(at 314.96 95.25)
+	)
+	(no_connect
 		(at 200.66 180.34)
 	)
 	(no_connect
+		(at 370.84 80.01)
+	)
+	(no_connect
 		(at 180.34 177.8)
 	)
@@
 	)
 	(no_connect
+		(at 370.84 121.92)
+	)
+	(no_connect
 		(at 200.66 177.8)
 	)
@@
 	)
 	(no_connect
+		(at 370.84 129.54)
+	)
+	(no_connect
+		(at 314.96 85.09)
+	)
+	(no_connect
 		(at 180.34 182.88)
 	)
@@
 	)
 	(no_connect
+		(at 370.84 110.49)
+	)
+	(no_connect
 		(at 180.34 180.34)
 	)
 	(no_connect
+		(at 314.96 121.92)
+	)
+	(no_connect
 		(at 200.66 182.88)
 	)
@@
 	)
 	(no_connect
+		(at 370.84 106.68)
+	)
+	(no_connect
+		(at 314.96 90.17)
+	)
+	(no_connect
 		(at 180.34 187.96)
 	)
 	(no_connect
+		(at 314.96 114.3)
+	)
+	(no_connect
 		(at 200.66 187.96)
 	)
 	(no_connect
+		(at 370.84 90.17)
+	)
+	(no_connect
+		(at 314.96 125.73)
+	)
+	(no_connect
+		(at 314.96 129.54)
+	)
+	(no_connect
 		(at 349.123 180.721)
 	)
+	(no_connect
+		(at 370.84 95.25)
+	)
 	(wire
 		(pts
@@
 	(wire
 		(pts
+			(xy 346.71 236.22) (xy 350.52 236.22)
+		)
+		(stroke
+			(width 0)
+			(type default)
+		)
+	)
+	(wire
+		(pts
+			(xy 334.01 233.68) (xy 346.71 233.68)
+		)
+		(stroke
+			(width 0)
+			(type default)
+		)
+	)
+	(wire
+		(pts
 			(xy 237.49 170.18) (xy 237.49 158.75)
 		)
@@
 	(wire
 		(pts
+			(xy 346.71 233.68) (xy 346.71 236.22)
+		)
+		(stroke
+			(width 0)
+			(type default)
+		)
+	)
+	(wire
+		(pts
 			(xy 321.31 224.79) (xy 321.31 224.663)
 		)
@@
 	(wire
 		(pts
+			(xy 334.01 233.68) (xy 334.01 235.458)
+		)
+		(stroke
+			(width 0)
+			(type default)
+		)
+	)
+	(wire
+		(pts
 			(xy 314.96 137.16) (xy 303.53 137.16)
 		)
@@
 	(wire
 		(pts
-			(xy 334.01 232.41) (xy 334.01 235.458)
+			(xy 334.01 232.41) (xy 334.01 233.68)
 		)
 		(stroke
@@
 	(wire
 		(pts
+			(xy 350.52 236.22) (xy 350.52 234.95)
+		)
+		(stroke
+			(width 0)
+			(type default)
+		)
+	)
+	(wire
+		(pts
 			(xy 212.09 82.55) (xy 229.87 82.55)
 		)
@@
 					(unit 1)
 				)
+			)
+		)
+	)
+	(symbol
+		(lib_id "Connector:TestPoint")
+		(at 350.52 234.95 0)
+		(unit 1)
+		(exclude_from_sim no)
+		(in_bom yes)
+		(on_board yes)
+		(dnp no)
+		(fields_autoplaced yes)
+		(property "Reference" "TP1"
+			(at 351.917 230.4358 0)
+			(effects
+				(font
+					(size 1.27 1.27)
+				)
+				(justify left)
+			)
+		)
+		(property "Value" "TestPoint"
+			(at 351.917 232.8601 0)
+			(effects
+				(font
+					(size 1.27 1.27)
+				)
+				(justify left)
+			)
+		)
+		(property "Footprint" "TestPoint:TestPoint_Keystone_5019_Miniature"
+			(at 355.6 234.95 0)
+			(effects
+				(font
+					(size 1.27 1.27)
+				)
+				(hide yes)
+			)
+		)
+		(property "Datasheet" "~"
+			(at 355.6 234.95 0)
+			(effects
+				(font
+					(size 1.27 1.27)
+				)
+				(hide yes)
+			)
+		)
+		(property "Description" "test point"
+			(at 350.52 234.95 0)
+			(effects
+				(font
+					(size 1.27 1.27)
+				)
+				(hide yes)
+			)
+		)
+		(pin "1"
+		)
+		(instances
+			(project ""
+				(path "/00ea9009-1039-4827-8fe4-64ceea0f3b86"
+					(reference "TP1")
+					(unit 1)
+				)

Commit message: feat: missed-cycle catch-up + PCB connector adjustment + test automation spec
Scheduler: a cycle whose scheduled start fell entirely within a power
outage (device down before AND after the trigger minute) was
previously skipped for the day with no catch-up -- checkPowerRecovery()
only resumes an already-running cycle, and the exact-minute trigger has
no memory of a missed minute. Added missed-cycle catch-up: on boot, any
enabled cycle whose start time has already passed today and hasn't run
since that scheduled time gets started now, for its full configured
duration/target, same as an on-time start.

Fixed two interaction bugs found while testing this on real hardware:
(1) catching up during begin() raced ahead of checkPowerRecovery(),
so a genuinely mid-run cycle interrupted by a second outage got
restarted from zero instead of resumed -- reordered so resume always
gets first refusal, with defensive guards on both sides; (2) the
catch-up check was keyed on any history entry for this cycle today,
so a cycle rescheduled to a new time after already running once earlier
the same day was wrongly skipped -- now anchored on history since the
cycle's CURRENT scheduled time specifically. Also restored an immediate
schedule check right after boot recovery, using the RTC's own time,
instead of waiting on the full WiFi/NTP/MQTT sequence to complete --
matters most exactly when it's needed most, since a power outage often
takes the router down too.

Hardware: adjusted connector position on Nursary_OneCH PCB (gerbers +
KiCad project regenerated) -- Avinash to test fit on his unit.

Added FG1 test jig specification (docs/testing/TEST_JIG_SPEC.md) and
a working Python test automation harness (products/FG1-flowguard/testing/)
-- flash + boot-log verification is usable today; production/full test
tiers are written against the jig's serial protocol, ready to wire up
once the physical jig exists.
Parts:
- D1, D4: footprint LED_0805_2012Metric -> Capacitor_SMD:C_1206_3216Metric
- D6: footprint Diode_SMD:D_SOD-882 -> Diode_SMD:D_0805_2012Metric
Changed lines of the file:
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@@
 			)
 		)
-		(property "Footprint" "LED_0805_2012Metric"
+		(property "Footprint" "Capacitor_SMD:C_1206_3216Metric"
 			(at 201.93 86.36 0)
 			(effects
@@
 			)
 		)
-		(property "Footprint" "LED_0805_2012Metric"
+		(property "Footprint" "Capacitor_SMD:C_1206_3216Metric"
 			(at 209.55 166.37 0)
 			(effects
@@
 			)
 		)
-		(property "Footprint" "Diode_SMD:D_SOD-882"
+		(property "Footprint" "Diode_SMD:D_0805_2012Metric"
 			(at 213.36 102.87 0)
 			(effects
