File: products/WPC-pumpcontroller/hardware/PumpNode/PumpNodeNew.kicad_sch (KiCad schematic)
At the start: 33 parts, among them J1 Conn_IN, J2 Conn_Coaxial_Small, J3 PWR_CONN, J4 Relay_CONN, K1 G6A, U1 ULN2003, U13 AMS1117-5.0, U5 ESP32 30 Pin CP2102 Developme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, U7 ISC-SX1262-B, U8 AP2112K-3.3

Commit message: WPC: update PumpNode/WPC/WPC-panel2x boards, regenerate fab outputs
- Update PumpNode, WPC, and WPC-panel2x KiCad PCB/schematic/project-local
  files
- Regenerate Gerber/drill exports for all three boards
- Add a separate fab_output/ Gerber set for WPC-panel2x alongside its
  existing GERBER-FLOW/ export
- Replace the old PumpNode/WPC-panel2x fab zip archives with freshly
  regenerated ones

Co-Authored-By: Claude Sonnet 5 <noreply@anthropic.com>
Parts:
- removed C4, C5: 220mfd,25V, Capacitor_THT:CP_Radial_D10.0mm_P2.50mm_P5.00mm, symbol Device:C_US
- removed H1: MountingHole, MountingHole:MountingHole_3.2mm_M3, symbol Mechanical:MountingHole
Connections:
- net RL1_CON_1: now also K1.14; no longer K1.24
- net RLY_COMM: now also K1.11; no longer K1.21
- net IN1_LED_MCU: no longer names the net of U5.22 (D33)
- net IN4_LED_MCU: no longer names the net of U5.28 (D13)
- no-connect marks 15 -> 17
