File: products/WPC-pumpcontroller/hardware/WPC-panel2x/WPC-panel2x.kicad_pcb (KiCad board)
At the start: 2 copper layers, 97.4 x 99.8 mm, 98 parts, among them J1 NoPWR_CONN, J2 Conn_Coaxial_Small, J3 PWR_CONN, J4 Conn_IN, U13 AMS1117-5.0, U5 ESP32 30 Pin CP2102 Developme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, U7 ISC-SX1262-B, U8 AP2112K-3.3

Commit message: WPC: update PumpNode/WPC/WPC-panel2x boards, regenerate fab outputs
- Update PumpNode, WPC, and WPC-panel2x KiCad PCB/schematic/project-local
  files
- Regenerate Gerber/drill exports for all three boards
- Add a separate fab_output/ Gerber set for WPC-panel2x alongside its
  existing GERBER-FLOW/ export
- Replace the old PumpNode/WPC-panel2x fab zip archives with freshly
  regenerated ones

Co-Authored-By: Claude Sonnet 5 <noreply@anthropic.com>
Parts:
- removed the . at (147.8, 73.0)
- removed the . at (103.3, 119.6)
- removed the . at (191.9, 54.0)
- removed the . at (147.5, 100.7)
- removed the . at (191.7, 119.6)
- removed the . at (103.5, 54.0)
- removed the C1 at (160.9, 104.9)
- removed the C1 at (134.3, 68.8)
- removed the C10 at (178.9, 68.2)
- removed the C10 at (116.4, 105.5)
- removed the C12 at (178.9, 78.4)
- removed the C12 at (116.4, 95.3)
- removed the C13 at (114.5, 95.3)
- removed the C13 at (180.7, 78.4)
- removed the C2 at (134.4, 71.3)
- removed the C2 at (160.8, 102.4)
- removed the C3 at (134.4, 73.8)
- removed the C3 at (160.9, 99.9)
- removed the C4 at (187.1, 64.3)
- removed the C4 at (108.2, 109.4)
- removed the C5 at (187.0, 75.0)
- removed the C5 at (108.2, 98.6)
- removed the C6 at (185.9, 39.9)
- removed the C6 at (109.3, 133.7)
- removed the C7 at (180.8, 68.2)
- removed the C7 at (114.4, 105.5)
- removed the C8 at (134.4, 66.2)
- removed the C8 at (160.9, 107.5)
- removed the D1 at (139.1, 120.9)
- removed the D1 at (156.1, 52.8)
- removed the D13 at (118.9, 101.3)
- removed the D13 at (176.4, 72.4)
- removed the D2 at (139.2, 107.8)
- removed the D2 at (156.1, 65.9)
- removed the D3 at (156.1, 79.0)
- removed the D3 at (139.2, 94.7)
- removed the D4 at (159.2, 48.2)
- removed the D4 at (136.1, 125.5)
- removed the D5 at (125.9, 125.5)
- removed the D5 at (169.3, 48.2)
- removed the D6 at (164.1, 48.1)
- removed the D6 at (131.1, 125.5)
- removed the D7 at (176.4, 61.9)
- removed the D7 at (118.9, 111.7)
- removed the D8 at (145.3, 48.2)
- removed the D8 at (149.9, 125.5)
- removed H1 (x2), H2 (x2), H4 (x2), H5 (x2): MountingHole, MountingHole:MountingHole_3.2mm_M3
- removed the J1 at (150.8, 43.9)
- removed the J1 at (144.5, 129.8)
- removed the J2 at (123.7, 90.3)
- removed the J2 at (171.5, 83.4)
- removed the J3 at (189.0, 43.8)
- removed the J3 at (106.3, 129.9)
- removed the J4 at (120.2, 129.9)
- removed the J4 at (175.0, 43.8)
- removed the R1 at (142.2, 94.7)
- removed the R1 at (153.0, 79.0)
- removed the R10 at (165.3, 102.4)
- removed the R10 at (129.9, 71.3)
- removed the R11 at (145.3, 51.4)
- removed the R11 at (149.9, 122.3)
- removed the R12 at (165.2, 107.6)
- removed the R12 at (130.1, 66.1)
- removed the R13 at (117.1, 58.5)
- removed the R13 at (178.1, 115.2)
- removed the R2 at (153.0, 65.9)
- removed the R2 at (142.2, 107.8)
- removed the R23 at (176.2, 68.0)
- removed the R23 at (119.0, 105.7)
- removed the R3 at (159.6, 51.4)
- removed the R3 at (135.7, 122.3)
- removed the R4 at (130.7, 122.2)
- removed the R4 at (164.5, 51.4)
- removed the R5 at (165.3, 104.9)
- removed the R5 at (129.9, 68.7)
- removed the R6 at (176.4, 57.8)
- removed the R6 at (118.9, 115.9)
- removed the R7 at (165.4, 100.0)
- removed the R7 at (129.9, 73.7)
- removed the R8 at (142.0, 121.0)
- removed the R8 at (153.2, 52.7)
- removed the R9 at (125.7, 122.3)
- removed the R9 at (169.6, 51.4)
- removed the U13 at (181.8, 57.8)
- removed the U13 at (113.4, 115.9)
- removed the U5 at (182.5, 132.9)
- removed the U5 at (112.8, 40.8)
- removed the U7 at (130.9, 104.4)
- removed the U7 at (164.3, 69.3)
- removed the U8 at (181.8, 73.5)
- removed the U8 at (113.4, 100.2)
- added .: MountingHole, MountingHole:MountingHole_3.2mm_M3, F.Cu at (99.0, 117.2)
- added .: MountingHole, MountingHole:MountingHole_3.2mm_M3, F.Cu at (54.6, 66.9)
- added .: MountingHole, MountingHole:MountingHole_3.2mm_M3, F.Cu at (143.2, 98.2)
- added .: MountingHole, MountingHole:MountingHole_3.2mm_M3, F.Cu at (98.7, 48.0)
- added .: MountingHole, MountingHole:MountingHole_3.2mm_M3, B.Cu at (54.8, 98.2)
- added .: MountingHole, MountingHole:MountingHole_3.2mm_M3, B.Cu at (143.0, 66.9)
- added C1: 100pF, Capacitor_SMD:C_0805_2012Metric, B.Cu at (112.2, 52.2)
- added C1: 100pF, Capacitor_SMD:C_0805_2012Metric, B.Cu at (85.6, 113.0)
- added C10: 10mfd,10V Tent, Capacitor_SMD:C_0805_2012Metric, B.Cu at (130.1, 112.4)
- added C10: 10mfd,10V Tent, Capacitor_SMD:C_0805_2012Metric, B.Cu at (67.6, 52.8)
- added C12: 10mfd,10V Tent, Capacitor_SMD:C_0805_2012Metric, B.Cu at (67.6, 42.6)
- added C12: 10mfd,10V Tent, Capacitor_SMD:C_0805_2012Metric, B.Cu at (130.1, 122.5)
- added C13: 100nF, Capacitor_SMD:C_0805_2012Metric, B.Cu at (132.0, 122.6)
- added C13: 100nF, Capacitor_SMD:C_0805_2012Metric, B.Cu at (65.8, 42.6)
- added C2: 100pF, Capacitor_SMD:C_0805_2012Metric, B.Cu at (85.6, 115.4)
- added C2: 100pF, Capacitor_SMD:C_0805_2012Metric, B.Cu at (112.1, 49.7)
- added C3: 100pF, Capacitor_SMD:C_0805_2012Metric, B.Cu at (112.1, 47.2)
- added C3: 100pF, Capacitor_SMD:C_0805_2012Metric, B.Cu at (85.6, 118.0)
- added C4: 1000mfd,25V, Capacitor_THT:CP_Radial_D10.0mm_P2.50mm_P5.00mm, F.Cu at (138.3, 108.5)
- added C4: 1000mfd,25V, Capacitor_THT:CP_Radial_D10.0mm_P2.50mm_P5.00mm, F.Cu at (59.4, 56.6)
- added C5: 1000mfd,25V, Capacitor_THT:CP_Radial_D10.0mm_P2.50mm_P5.00mm, F.Cu at (59.5, 45.9)
- added C5: 1000mfd,25V, Capacitor_THT:CP_Radial_D10.0mm_P2.50mm_P5.00mm, F.Cu at (138.3, 119.2)
- added C6: 100nF, Capacitor_SMD:C_0805_2012Metric, B.Cu at (60.3, 80.0)
- added C6: 100nF, Capacitor_SMD:C_0805_2012Metric, B.Cu at (137.4, 85.1)
- added C7: 100nF, Capacitor_SMD:C_0805_2012Metric, B.Cu at (132.0, 112.4)
- added C7: 100nF, Capacitor_SMD:C_0805_2012Metric, B.Cu at (65.7, 52.8)
- added C8: 100pF, Capacitor_SMD:C_0805_2012Metric, B.Cu at (85.6, 110.3)
- added C8: 100pF, Capacitor_SMD:C_0805_2012Metric, B.Cu at (112.1, 54.8)
- added D1: LED_GREEN_IN1, LED_SMD:LED_1206_3216Metric, F.Cu at (90.4, 68.2)
- added D1: LED_GREEN_IN1, LED_SMD:LED_1206_3216Metric, F.Cu at (107.3, 97.0)
- added D13: LED_Yellow_LoRa, LED_SMD:LED_1206_3216Metric, F.Cu at (127.6, 116.6)
- added D13: LED_Yellow_LoRa, LED_SMD:LED_1206_3216Metric, F.Cu at (70.1, 48.5)
- added D2: LED_GREEN_IN2, LED_SMD:LED_1206_3216Metric, F.Cu at (90.4, 55.1)
- added D2: LED_GREEN_IN2, LED_SMD:LED_1206_3216Metric, F.Cu at (107.3, 110.1)
- added D3: LED_GREEN_IN3, LED_SMD:LED_1206_3216Metric, F.Cu at (107.3, 123.2)
- added D3: LED_GREEN_IN3, LED_SMD:LED_1206_3216Metric, F.Cu at (90.4, 42.0)
- added D4: PESD3V3U1UL, Diode_SMD:D_0603_1608Metric, B.Cu at (87.3, 72.8)
- added D4: PESD3V3U1UL, Diode_SMD:D_0603_1608Metric, B.Cu at (110.4, 92.4)
- added D5: PESD3V3U1UL, Diode_SMD:D_0603_1608Metric, B.Cu at (77.2, 72.8)
- added D5: PESD3V3U1UL, Diode_SMD:D_0603_1608Metric, B.Cu at (120.5, 92.4)
- added D6: PESD3V3U1UL, Diode_SMD:D_0603_1608Metric, B.Cu at (115.4, 92.3)
- added D6: PESD3V3U1UL, Diode_SMD:D_0603_1608Metric, B.Cu at (82.4, 72.8)
- added D7: LED_RED_IN4, LED_SMD:LED_1206_3216Metric, F.Cu at (127.6, 106.1)
- added D7: LED_RED_IN4, LED_SMD:LED_1206_3216Metric, F.Cu at (70.1, 59.0)
- added D8: PESD3V3U1UL, Diode_SMD:D_0603_1608Metric, B.Cu at (101.2, 72.8)
- added D8: PESD3V3U1UL, Diode_SMD:D_0603_1608Metric, B.Cu at (96.5, 92.3)
- added J1: NoPWR_CONN, Connector_Phoenix_MSTB:PhoenixContact_MSTBA_2,5_2-G-5,08_1x02_P5.08mm_Horizontal, F.Cu at (95.7, 77.1)
- added J1: NoPWR_CONN, Connector_Phoenix_MSTB:PhoenixContact_MSTBA_2,5_2-G-5,08_1x02_P5.08mm_Horizontal, F.Cu at (102.0, 88.1)
- added J2: Conn_Coaxial_Small, Connector_Coaxial:SMA_Samtec_SMA-J-P-H-ST-EM1_EdgeMount, B.Cu at (122.8, 127.1)
- added J2: Conn_Coaxial_Small, Connector_Coaxial:SMA_Samtec_SMA-J-P-H-ST-EM1_EdgeMount, B.Cu at (75.0, 38.0)
- added J3: PWR_CONN, Connector_Phoenix_MSTB:PhoenixContact_MSTBA_2,5_2-G-5,08_1x02_P5.08mm_Horizontal, F.Cu at (57.5, 77.2)
- added J3: PWR_CONN, Connector_Phoenix_MSTB:PhoenixContact_MSTBA_2,5_2-G-5,08_1x02_P5.08mm_Horizontal, F.Cu at (140.2, 88.0)
- added J4: Conn_IN, Connector_Phoenix_MSTB:PhoenixContact_MSTBA_2,5_4-G-5,08_1x04_P5.08mm_Horizontal, F.Cu at (126.2, 88.0)
- added J4: Conn_IN, Connector_Phoenix_MSTB:PhoenixContact_MSTBA_2,5_4-G-5,08_1x04_P5.08mm_Horizontal, F.Cu at (71.5, 77.2)
- added R1: 470E, Resistor_SMD:R_0805_2012Metric, B.Cu at (93.5, 42.0)
- added R1: 470E, Resistor_SMD:R_0805_2012Metric, B.Cu at (104.2, 123.2)
- added R10: 10K, Resistor_SMD:R_0805_2012Metric, B.Cu at (81.1, 115.5)
- added R10: 10K, Resistor_SMD:R_0805_2012Metric, B.Cu at (116.6, 49.6)
- added R11: 470E, Resistor_SMD:R_0805_2012Metric, B.Cu at (101.2, 69.5)
- added R11: 470E, Resistor_SMD:R_0805_2012Metric, B.Cu at (96.5, 95.6)
- added R12: 10K, Resistor_SMD:R_0805_2012Metric, B.Cu at (116.4, 54.9)
- added R12: 10K, Resistor_SMD:R_0805_2012Metric, B.Cu at (81.3, 110.3)
- added R13: 10K, Resistor_SMD:R_0805_2012Metric, B.Cu at (68.3, 102.7)
- added R13: 10K, Resistor_SMD:R_0805_2012Metric, B.Cu at (129.4, 62.5)
- added R2: 470E, Resistor_SMD:R_0805_2012Metric, B.Cu at (104.2, 110.1)
- added R2: 470E, Resistor_SMD:R_0805_2012Metric, B.Cu at (93.5, 55.0)
- added R23: 470E, Resistor_SMD:R_0805_2012Metric, B.Cu at (127.4, 112.2)
- added R23: 470E, Resistor_SMD:R_0805_2012Metric, B.Cu at (70.3, 53.0)
- added R3: 470E, Resistor_SMD:R_0805_2012Metric, B.Cu at (86.9, 69.6)
- added R3: 470E, Resistor_SMD:R_0805_2012Metric, B.Cu at (110.8, 95.6)
- added R4: 470E, Resistor_SMD:R_0805_2012Metric, B.Cu at (115.8, 95.6)
- added R4: 470E, Resistor_SMD:R_0805_2012Metric, B.Cu at (82.0, 69.5)
- added R5: 10K, Resistor_SMD:R_0805_2012Metric, B.Cu at (81.2, 112.9)
- added R5: 10K, Resistor_SMD:R_0805_2012Metric, B.Cu at (116.6, 52.2)
- added R6: 470E, Resistor_SMD:R_0805_2012Metric, B.Cu at (127.6, 101.9)
- added R6: 470E, Resistor_SMD:R_0805_2012Metric, B.Cu at (70.1, 63.2)
- added R7: 10K, Resistor_SMD:R_0805_2012Metric, B.Cu at (116.6, 47.2)
- added R7: 10K, Resistor_SMD:R_0805_2012Metric, B.Cu at (81.1, 117.9)
- added R8: 470E, Resistor_SMD:R_0805_2012Metric, B.Cu at (93.3, 68.3)
- added R8: 470E, Resistor_SMD:R_0805_2012Metric, B.Cu at (104.4, 96.9)
- added R9: 470E, Resistor_SMD:R_0805_2012Metric, B.Cu at (76.9, 69.6)
- added R9: 470E, Resistor_SMD:R_0805_2012Metric, B.Cu at (120.8, 95.6)
- added U13: AMS1117-5.0, Package_TO_SOT_SMD:SOT-223-3_TabPin2, B.Cu at (64.7, 63.1)
- added U13: AMS1117-5.0, Package_TO_SOT_SMD:SOT-223-3_TabPin2, B.Cu at (133.1, 102.0)
- added U5: ESP32 30 Pin CP2102 Development Board, PCM_Espressif:ESP32-C3-DevKitM-1, F.Cu at (133.7, 80.2)
- added U5: ESP32 30 Pin CP2102 Development Board, PCM_Espressif:ESP32-C3-DevKitM-1, F.Cu at (64.0, 85.0)
- added U7: ISC-SX1262-B, RF_Module:Ai-Thinker-Ra-01-LoRa, B.Cu at (82.2, 51.7)
- added U7: ISC-SX1262-B, RF_Module:Ai-Thinker-Ra-01-LoRa, B.Cu at (115.6, 113.5)
- added U8: AP2112K-3.3, Package_TO_SOT_SMD:SOT-23-5, B.Cu at (64.7, 47.5)
- added U8: AP2112K-3.3, Package_TO_SOT_SMD:SOT-23-5, B.Cu at (133.1, 117.7)
Routing:
- net +5V: track 190.6 -> 202.6 mm, vias 0 -> 14
- net +8V: track 62.2 -> 59.4 mm
- net /NSS: track 213.9 -> 213.3 mm
Other:
- board size 97.4 x 99.8 mm -> 95.5 x 93.4 mm
