File: products/WM2-watermaster/hardware/SolarNode/WM2-SolarNode.kicad_sch (KiCad schematic)
At the start: 77 parts, among them J1 SOLAR_12V_IN (screw terminal), J10 VALVE1, J11 VALVE2, J2 USB-C (program/console), J3 PUMP1 field wiring (verify NO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, J4 PUMP2 field wiring (verify NO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, J5 FLOW1 (VCC/GND/Signal), J6 FLOW2 (VCC/GND/Signal), J7 FLOW3 (VCC/GND/Signal), J8 FLOW4 (VCC/GND/Signal), J9 PRESSURE1, K1 SRD-05VDC-SL-C, K2 SRD-05VDC-SL-C, SW1 RESET (EN), SW2 BOOT (shared w/ I2C_SCL; hold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, U1 AP63205WU (fixed 5.0V out), U2 AP2112K-3.3, U3 ESP32-C3-WROOM-02, U4 DS1307Z+, U5 ULN2003, U6 DRV8871DDA, U7 DRV8871DDA, Y1 32.768kHz

Commit message: Workshop labs page at /workshop, GPSIOAM workshop materials, pending WIP
- agrisense-webapp: public, no-login /workshop route (middleware allowlist +
  next.config.ts rewrite) serving the student labs page from public/workshop
- docs/workshops/gpsioam-2026: 4 Wokwi-ready ESP32 labs + Lab 4 reference
  solution, labs page template and build_site.py
- Pending work committed as-is: WM2 SolarNode/WaterMaster KiCad, WPC Pump
  Node Gerbers, FG1 flash tools, marketing video projects
- .gitignore: Next.js cache, *.tsbuildinfo, KiCad *.lck, .claude/settings.local.json;
  stop tracking .next/cache

Co-Authored-By: Claude Opus 5.5 <noreply@anthropic.com>
Parts:
- renumbered LED8A to LED8A1, LED8B to LED8B1, LED9A to LED9A1, LED9B to LED9B1
Connections:
- net PROT_A is gone; now on net +12V: D1.2 (A), F1.2
- no-connect marks 16 -> 13
Other:
- moved on the sheet: C3, F1, J2, U2, U3
