File: products/WM2-watermaster/hardware/WaterMaster/WM2-WaterMaster.kicad_sch (KiCad schematic)
At the start: 106 parts, among them J1 Flow_CONN, J12 Conn_01x04_Pin, J13 Conn_01x03_Pin, J2 Conn_Coaxial_Small, J3 PWR_CONN, J4 Conn_IN, J5 Conn_01x03_Pin, J7 Conn_RLY_EXTENDER, K1 Cube_Relay, K2 Cube_Relay, K3 Cube_Relay, K4 Cube_Relay, K5 Cube_Relay, K6 Cube_Relay, U1 ULN2003, U10 DS1307Z+, U13 AMS1117-5.0, U2 74HC595, U3 MT3608, U4 DS3231M, U5 ESP32 30 Pin CP2102 Developme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, U7 ISC-SX1262-B, U8 AP2112K-3.3, U9 74HC595, Y1 Crystal

Commit message: Workshop labs page at /workshop, GPSIOAM workshop materials, pending WIP
- agrisense-webapp: public, no-login /workshop route (middleware allowlist +
  next.config.ts rewrite) serving the student labs page from public/workshop
- docs/workshops/gpsioam-2026: 4 Wokwi-ready ESP32 labs + Lab 4 reference
  solution, labs page template and build_site.py
- Pending work committed as-is: WM2 SolarNode/WaterMaster KiCad, WPC Pump
  Node Gerbers, FG1 flash tools, marketing video projects
- .gitignore: Next.js cache, *.tsbuildinfo, KiCad *.lck, .claude/settings.local.json;
  stop tracking .next/cache

Co-Authored-By: Claude Opus 5.5 <noreply@anthropic.com>
Parts:
- removed C1, C13, C15, C17, C18, C2, C7: 100nF, Capacitor_SMD:C_0805_2012Metric, symbol Device:C
- removed C12: 10mfd,10V tentalum, Capacitor_SMD:C_0603_1608Metric, symbol Device:C_US
- removed C16: 1000uF,25V, Capacitor_THT:CP_Radial_D10.0mm_P2.50mm_P5.00mm, symbol Device:C_US
- removed C20, C21: 100pF, Capacitor_SMD:C_0805_2012Metric, symbol Device:C
- removed C22: 22µF, X7R, 35V,1210, Capacitor_SMD:C_0805_2012Metric, symbol Device:C
- removed C4, C5: 1000mfd,25V, Capacitor_THT:CP_Radial_D10.0mm_P2.50mm_P5.00mm, symbol Device:C_US
- removed C?: 10Mfd, Capacitor_SMD:C_0805_2012Metric, symbol Device:C
- removed D13: LED_Yellow_LoRa, LED_SMD:LED_0805_2012Metric_Pad1.15x1.40mm_HandSolder, symbol Device:LED
- removed D14, D15: LED_YELLOW_PUMP, LED_SMD:LED_0805_2012Metric_Pad1.15x1.40mm_HandSolder, symbol Device:LED
- removed D16, D17, D18, D19, D5, D6, D8: PESD3V3U1UL, Diode_SMD:D_SOD-882, symbol Diode:PESD3V3U1UL
- removed D2: LED_GREEN_IN2, LED_SMD:LED_0805_2012Metric_Pad1.15x1.40mm_HandSolder, symbol Device:LED
- removed D20: LED_Green_PR1, LED_SMD:LED_0805_2012Metric_Pad1.15x1.40mm_HandSolder, symbol Device:LED
- removed D21: LED_Green_PR2, LED_SMD:LED_0805_2012Metric_Pad1.15x1.40mm_HandSolder, symbol Device:LED
- removed D22: LED_R_LoBAT, LED_SMD:LED_0805_2012Metric_Pad1.15x1.40mm_HandSolder, symbol Device:LED
- removed D9: SS34, Diode_SMD:D_SMA, symbol Diode:SS34
- removed J12: Conn_01x04_Pin, Connector_Phoenix_MSTB:PhoenixContact_MSTBA_2,5_4-G-5,08_1x04_P5.08mm_Horizontal, symbol Connector:Conn_01x04_Pin
- removed J13: Conn_01x03_Pin, Connector_Phoenix_MSTB:PhoenixContact_MSTBA_2,5_3-G-5,08_1x03_P5.08mm_Horizontal, symbol Connector:Conn_01x03_Pin
- removed J2: Conn_Coaxial_Small, Connector_Coaxial:SMA_Samtec_SMA-J-P-H-ST-EM1_EdgeMount, symbol Connector:Conn_Coaxial_Small
- removed J3: PWR_CONN, Connector_Phoenix_MSTB:PhoenixContact_MSTBVA_2,5_2-G-5,08_1x02_P5.08mm_Vertical, symbol Connector:Conn_01x02_Pin
- removed J4: Conn_IN, Connector_Phoenix_MSTB:PhoenixContact_MSTBA_2,5_4-G-5,08_1x04_P5.08mm_Horizontal, symbol Connector:Conn_01x04_Pin
- removed J7: Conn_RLY_EXTENDER, Connector_Phoenix_MSTB:PhoenixContact_MSTBVA_2,5_4-G-5,08_1x04_P5.08mm_Vertical, symbol Connector:Conn_01x04_Pin
- removed K1, K2, K3, K4, K5, K6: Cube_Relay, Relay_THT:Relay_SPDT_SANYOU_SRD_Series_Form_C, symbol Relay:SANYOU_SRD_Form_C
- removed R1, R2, R23, R28, R29, R30, R31: 470E, Resistor_SMD:R_0805_2012Metric, symbol Device:R
- removed R24, R25: 1K, Resistor_SMD:R_0805_2012Metric, symbol Device:R
- removed R26, R27: 150E,1%, Resistor_SMD:R_0805_2012Metric, symbol Device:R
- removed R?: 100K, Resistor_SMD:R_0805_2012Metric, symbol Device:R
- removed U1: ULN2003, Package_SO:SOIC-16_3.9x9.9mm_P1.27mm, symbol Transistor_Array:ULN2003
- removed U13: AMS1117-5.0, Package_TO_SOT_SMD:SOT-223-3_TabPin2, symbol Regulator_Linear:AMS1117-5.0
- removed U2, U9: 74HC595, Package_SO:SOIC-16_3.9x9.9mm_P1.27mm, symbol 74xx:74HC595
- removed U3: MT3608, Package_TO_SOT_SMD:SOT-23-6, symbol Regulator_Switching:MT3608
- removed U4: DS3231M, Package_SO:SOIC-16W_7.5x10.3mm_P1.27mm, symbol Timer_RTC:DS3231M
- removed U5: ESP32 30 Pin CP2102 Development Board, PCM_Espressif:ESP32-C3-DevKitM-1, symbol PCM_Espressif:ESP32-C3-DevKitM-1
- removed U7: ISC-SX1262-B, RF_Module:ISC-LoRa, symbol RF_Module:Ai-Thinker-Ra-01
- removed U8: AP2112K-3.3, Package_TO_SOT_SMD:SOT-23-5, symbol Regulator_Linear:AP2112K-3.3
- added C12: 100nF, Capacitor_SMD:C_0805_2012Metric, symbol Device:C
- added C13, C15: 22uF/16V, Capacitor_SMD:C_0805_2012Metric, symbol Device:C_US
- added C17: 10mfd,10V tent, Capacitor_SMD:C_0805_2012Metric, symbol Device:C_US
- added C18: 10,10V tent, Capacitor_SMD:C_0805_2012Metric, symbol Device:C_US
- added C3, C4, C5: 100pF, Capacitor_SMD:C_0805_2012Metric, symbol Device:C
- added C7, C9: 1000mfd,25V, Capacitor_THT:CP_Radial_D10.0mm_P2.50mm_P5.00mm, symbol Device:C_US
- added C8: 10uF/25V, Capacitor_SMD:C_0805_2012Metric, symbol Device:C_US
- added D5: LED_Green_Flow, Capacitor_SMD:C_1206_3216Metric, symbol Device:LED
- added D6: SS34 (reverse-polarity), Diode_SMD:D_SMA, symbol Diode:SS34
- added D7: LED_G_PWR, Capacitor_SMD:C_1206_3216Metric, symbol Device:LED
- added D8: LED_V1_Green, Capacitor_SMD:C_1206_3216Metric, symbol Device:LED
- added D9: LED_V2_Green, Capacitor_SMD:C_1206_3216Metric, symbol Device:LED
- added F3: Polyfuse_Small, Inductor_SMD:L_1206_3216Metric, symbol Device:Polyfuse_Small
- added H1, H2, H3, H4, H5: MountingHole, MountingHole:MountingHole_4.5mm, symbol Mechanical:MountingHole
- added J2, J3, J4: Flow_Conn, Connector_Phoenix_MSTB:PhoenixContact_MSTBVA_2,5_3-G-5,08_1x03_P5.08mm_Vertical, symbol Connector:Conn_01x03_Pin
- added J6: SOLAR_12V_IN, Connector_Phoenix_MSTB:PhoenixContact_MSTBA_2,5_2-G-5,08_1x02_P5.08mm_Horizontal, symbol Connector:Conn_01x02_Pin
- added J7, J8: LV_Conn, Connector_Phoenix_MSTB:PhoenixContact_MSTBA_2,5_2-G-5,08_1x02_P5.08mm_Horizontal, symbol Connector:Conn_01x02_Pin
- added J9: Programmer_Conn, Connector_JST:JST_XH_B8B-XH-AM_1x08_P2.50mm_Vertical, symbol Connector:Conn_01x08_Socket
- added R15: 10K, Resistor_SMD:R_0805_2012Metric, symbol Device:R
- added R16: 22K, Resistor_SMD:R_0805_2012Metric, symbol Device:R
- added R18, R19, R8, R9: 470E, Resistor_SMD:R_0805_2012Metric, symbol Device:R
- added SW1: RESET (EN), Button_Switch_SMD:SW_Tactile_SPST_NO_Straight_CK_PTS636Sx25SMTRLFS, symbol Switch:SW_Push
- added U1, U2: DRV8871DDA, Package_SO:Texas_HTSOP-8-1EP_3.9x4.9mm_P1.27mm_EP2.95x4.9mm_Mask2.4x3.1mm_ThermalVias, symbol Driver_Motor:DRV8871DDA
- added U3: AP63205WU (fixed 5.0V out), Package_TO_SOT_SMD:TSOT-23-6, symbol Regulator_Switching:AP63205WU
- added U4: ESP32-WROOM-32D, RF_Module:ESP32-WROOM-32D, symbol RF_Module:ESP32-WROOM-32D
- added U6: AP2112K-3.3, Package_TO_SOT_SMD:SOT-23-5, symbol Regulator_Linear:AP2112K-3.3
- C10: value 10mfd,10V tentalum -> 1000mfd,25V; footprint Capacitor_SMD:C_0603_1608Metric -> Capacitor_THT:CP_Radial_D10.0mm_P2.50mm_P5.00mm
- C14: value 22µF, X7R,35V,1210 -> 100nF
- D1: value LED_GREEN_IN1 -> LED_GREEN_PS; footprint LED_SMD:LED_0805_2012Metric_Pad1.15x1.40mm_HandSolder -> Capacitor_SMD:C_1206_3216Metric
- D10: value LED_YELLOW_PUMP -> LED_V1_Yellow; footprint LED_SMD:LED_0805_2012Metric_Pad1.15x1.40mm_HandSolder -> Capacitor_SMD:C_1206_3216Metric
- D11: value LED_YELLOW_PUMP -> LED_V2_Yellow; footprint LED_SMD:LED_0805_2012Metric_Pad1.15x1.40mm_HandSolder -> Capacitor_SMD:C_1206_3216Metric
- D12: value LED_YELLOW_PUMP -> LED_B_WIFI; footprint LED_SMD:LED_0805_2012Metric_Pad1.15x1.40mm_HandSolder -> Capacitor_SMD:C_1206_3216Metric
- D2: renamed from D7; footprint LED_SMD:LED_0805_2012Metric_Pad1.15x1.40mm_HandSolder -> Capacitor_SMD:C_1206_3216Metric
- D3: value LED_GREEN_IN3 -> LED_Green_Flow; footprint LED_SMD:LED_0805_2012Metric_Pad1.15x1.40mm_HandSolder -> Capacitor_SMD:C_1206_3216Metric
- D4: value LED_YELLOW_PUMP -> LED_Green_Flow; footprint LED_SMD:LED_0805_2012Metric_Pad1.15x1.40mm_HandSolder -> Capacitor_SMD:C_1206_3216Metric
- F1, F2: value Polyfuse_Small -> 500mA
- J1: value Flow_CONN -> Press_Conn; footprint PhoenixContact_MSTBA_2,5_2-G-5,08_1x02_P5.08mm_Horizontal -> Connector_Phoenix_MSTB:PhoenixContact_MSTBA_2,5_2-G-5,08_1x02_P5.08mm_Horizontal
- J5: value Conn_01x03_Pin -> Flow_Conn; footprint Connector_Phoenix_MSTB:PhoenixContact_MSTBA_2,5_3-G-5,08_1x03_P5.08mm_Horizontal -> Connector_Phoenix_MSTB:PhoenixContact_MSTBVA_2,5_3-G-5,08_1x03_P5.08mm_Vertical
- L1: value 10microH -> 4.7uH; footprint Inductor_SMD:L_6.3x6.3_H3 -> Inductor_SMD:L_Neosid_Ms85T
- R14: value 324K,1% -> 10K
- R17: value 10K,1% -> 22K
- R20, R22, R5: value 1K -> 470E
- R21: value 1K -> 10K
- Y1: footprint Crystal:Crystal_AT310_D3.0mm_L10.0mm_Horizontal -> Crystal_C38-LF_D3.0mm_L8.0mm_Horizontal
- renumbered C3 to C1, C19 to C16, C8 to C2, R8 to R1, R7 to R11, R6 to R2, R18 to R23, R32 to R24, R33 to R25, R15 to R26, R16 to R27, R9 to R6, R11 to R7, U10 to U5
Connections:
- net IN1_CON is gone; now on an unnamed net: R6.2
- net IN3_CON is gone; now on an unnamed net: R3.2
- net Press_IN1_CON is gone; now on an unnamed net: J5.2 (Pin_2)
- net Press_IN2_CON is gone; now on net GND: J5.3 (Pin_3)
- net RELAY1_COIL is gone; now on net GND: D4.1 (K)
- net RELAY4_COIL is gone; now on net GND: D12.1 (K)
- net +3.3V: now also C14.1, R14.1, R21.1, C18.1, R15.1, U4.2 (VDD), U6.5 (VOUT); no longer C11.1
- net +5V: now also L1.2, C13.1, C15.1, C17.1, F3.1, J9.8 (Pin_8), U3.1 (FB), U6.1 (VIN), U6.3 (EN); no longer C10.1, F2.1
- net Batt_Mon: now also U4.9 (IO33)
- net GND: now also C13.2, C15.2, C17.2, C18.2, C3.2, C4.2, C5.2, C7.2, C8.2, C9.2, D5.1 (K), D7.1 (K), J2.3 (Pin_3), J3.3 (Pin_3), J4.3 (Pin_3), J6.1 (Pin_1), J9.4 (Pin_4), J9.7 (Pin_7), R16.2, SW1.2, U1.1 (GND), U1.7 (GND), U1.9 (GND), U2.1 (GND), U2.7 (GND), U2.9 (GND), U3.4 (GND), U4.1 (GND), U4.15 (GND), U4.38 (GND), U4.39 (GND), U6.2 (GND)
- net SCL: now also U4.36 (IO22)
- net SDA: now also U4.33 (IO21)
- net at R5.2: now also D5.2 (A); no longer D4.2 (A)
- net at D10.2 (A): now also D8.1 (K), R19.2; no longer R20.2
- net at R17.1: now also U2.4 (ILIM); no longer R14.2
- net at D11.2 (A): now also R20.2, D9.1 (K); no longer R21.2
- net +20V renamed +12V
- net +12V: now also C6.1, R23.1, C8.1, D6.1 (K), R18.1, U3.2 (EN), U3.3 (IN); no longer R14.1
- net +20VPR renamed +12V_LV
- net +12V_LV: now also C10.1, C7.1, C9.1, U1.5 (VM), U2.5 (VM); no longer J5.1 (Pin_1)
- removed net +5VR: F2.2, R20.1, R21.1, R22.1, R5.1
- removed net +8V: C14.1, C6.1, L1.1, R23.1
- net Flow_CON: no longer names the net of J1.2 (Pin_2)
- net Flow_CON: no longer R7.2
- net Flow_LED renamed Flow_LED1
- net Flow_LED1: now also U4.10 (IO25)
- net Flow_MCU renamed Flow_MCU1
- net Flow_MCU1: now also U4.6 (IO34)
- net IN1 renamed PS_MCU
- net PS_MCU: now also U4.8 (IO32)
- net IN1_LED renamed PS_LED
- net PS_LED: now also U4.12 (IO27)
- net IN2 renamed Flow_LED4
- net Flow_LED4: now also U4.30 (IO18)
- net IN2_CON: no longer names the net of R4.2
- net IN2_CON: now also D4.2 (A)
- net IN3 renamed Flow_LED3
- net Flow_LED3: now also U4.31 (IO19)
- net LOBATT_LED renamed Flow_MCU2
- net Flow_MCU2: now also C5.1, R15.2, U4.7 (IO35)
- net NSS renamed Flow_MCU3
- net Flow_MCU3: now also C3.1, R8.1, U4.4 (IO36/SENSOR_VP)
- net RELAY2_COIL renamed V1_OUT2
- net V1_OUT2: now also D8.2 (A), J7.2 (Pin_2), U1.8 (OUT2)
- net RELAY3_COIL renamed V2_OUT2
- net V2_OUT2: now also D9.2 (A), J8.2 (Pin_2), U2.8 (OUT2)
- new net: D6.2 (A), F2.2
- new net: J3.2 (Pin_2), R8.2
- new net: C12.2, L1.1, U3.5 (SW)
- new net: J4.2 (Pin_2), R9.2
- new net: F2.1, J6.2 (Pin_2)
- new net: D7.2 (A), R18.2
- new net: R16.1, U1.4 (ILIM)
- new net: C12.1, U3.6 (BST)
- new net: J2.2 (Pin_2), R7.2
- new net +5V_Ext: F3.2, J2.1 (Pin_1), J3.1 (Pin_1), J4.1 (Pin_1), J5.1 (Pin_1)
- new net EN: C11.1, J9.5 (Pin_5), R21.2, SW1.1, U4.3 (EN)
- new net Flow_LED2: R5.1, U4.11 (IO26)
- new net Flow_MCU4: C4.1, R14.2, R9.1, U4.5 (IO39/SENSOR_VN)
- new net IO0: J9.6 (Pin_6), U4.25 (IO0)
- new net LV1_IN1_MCU: U1.3 (IN1), U4.16 (IO13)
- new net LV1_IN2_MCU: U1.2 (IN2), U4.26 (IO4)
- new net LV2_IN1_MCU: U2.3 (IN1), U4.27 (IO16)
- new net LV2_IN2_MCU: U2.2 (IN2), U4.28 (IO17)
- new net RXD0: J9.2 (Pin_2), U4.34 (RXD0/IO3)
- new net TXD0: J9.3 (Pin_3), U4.35 (TXD0/IO1)
- new net V1_OUT1: J7.1 (Pin_1), R19.1, U1.6 (OUT1)
- new net V2_OUT1: J8.1 (Pin_1), R20.1, U2.6 (OUT1)
- new net WIFI_LED: R22.1, U4.13 (IO14)
- no-connect marks 18 -> 13
Other:
- note added: "5V to 3.3V"
- note added: "Batt Monitoring"
- note added: "ESP32"
- note added: "F1"
- note added: "F2"
- note added: "F3"
- note added: "F4"
- note added: "INPUT POWER +12V"
- note added: "Latch Valve"
- note added: "Pressure Switch"
- note removed: "ESP32 -30 pin Dev Kit"
- note removed: "FTDI USB-to-TTL adapter connected to the 6-pin header on the board's edge. The pinout alignment is typically: DTR, TXO, RXI, VCC, CTS, and GND. Key connections are DTR-to-DTR, TX-to-RXI, RX-to-TXO, VCC-to-VCC, and GND-to-GND"
- note removed: "IN1(D) No Power"
- note removed: "IN2(A)"
- note removed: "IN3(A)"
- note removed: "INPUT POWER +8V"
- note removed: "LoRa"
- note removed: "On Board LED as WiFi and Power LED"
- note removed: "Pressure Sensor INPUT(4-20ma)"
- note removed: "Programmer cum Debugger https://evelta.com/7semi-st-link-v2-v2-1-usb-c-debugger-programmer-for-stm32-mcus/ From the photo, the 7Semi ST‑Link V2 has this pin order (top to bottom on the right header): SWO RST SWDIO GND SWCLK 3V3 On your STM32G030 board, make a 6‑pin (or 5‑pin) header in the same order, and wire: SWO → optional (PB3, can be left NC for now) RST → NRST SWDIO → PA13 GND → GND SWCLK →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"
- note removed: "Put RC to delay the output of relay to avoid startup ON"
- note removed: "RL1"
- note removed: "RL2"
- note removed: "RL3"
- note removed: "RL4"
- note removed: "RL5"
- note removed: "RL6"
- note removed: "Valve CONTROL OUTPUT"
- note removed: "Voltage Booster"
- note removed: "X"
- moved on the sheet: BT1, C1, C16, D1, R1, R11, R23, R24, R25, R26, R27, R6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
