File: products/WM2-watermaster/hardware/WaterMaster/WM2-WaterMaster.kicad_sch (KiCad schematic)
At the start: 84 parts, among them J1 Press_Conn, J2 Flow_Conn, J3 Flow_Conn, J4 Flow_Conn, J5 Flow_Conn, J6 SOLAR_12V_IN, J7 LV_Conn, J8 LV_Conn, J9 Programmer_Conn, SW1 RESET (EN), U1 DRV8871DDA, U2 DRV8871DDA, U3 AP63205WU (fixed 5.0V out), U4 ESP32-WROOM-32D, U5 DS1307Z+, U6 AP2112K-3.3, Y1 Crystal

Commit message: WM2-WaterMaster: redesign for Girish Farm (ESP32-WROOM-32D, solar/battery)
Full schematic redesign of the WM2 main board, moving from the WM1-
copied ESP32-C3 devkit design to a bare ESP32-WROOM-32D module for
the extra GPIO headroom this deployment needs:

- 12V solar input -> AP63205WU buck (5V) -> AP2112K-3.3 LDO (3.3V)
- 4x flow sensor + 1x pressure switch inputs, each with a firmware-
  driven LED (stretched blink) on its own GPIO for field troubleshooting
- Battery voltage monitoring (resistor divider -> ADC)
- WiFi status LED
- 2x latch-valve driver (DRV8871) with anti-parallel LED pairs across
  OUT1/OUT2, catching both open and close pulses without spending a
  GPIO on it
- 2x relay-based valve control as an alternate/either-or population
  option, sharing the same MCU control nets as the latch drivers
- DS1307Z+ RTC with CR2032 backup
- 8-pin bare UART header (no onboard USB-UART chip) for one-time
  factory flashing via an external CP2102-based programmer with
  auto-reset (EN/IO0 driven by the programmer's own transistor
  circuit); all further updates go out over WiFi OTA

Also includes the first full PCB layout and regenerated gerbers/
production zip (WM2-Girish.zip, replacing the placeholder mini zip).

Co-Authored-By: Claude Sonnet 5 <noreply@anthropic.com>
Parts:
- C13, C15, C8: footprint Capacitor_SMD:C_0805_2012Metric -> Capacitor_SMD:C_1206_3216Metric_Pad1.33x1.80mm_HandSolder
- C17: value 10mfd,10V tent -> 10u/10V tent
- C18: value 10,10V tent -> 10u/10V tent
- D6: value SS34 (reverse-polarity) -> SS34
- U3: value AP63205WU (fixed 5.0V out) -> AP63205WU
- renumbered D7 to LD1, D9 to LD10, D11 to LD11, D12 to LD2, D2 to LD3, D5 to LD4, D3 to LD5, D4 to LD6, D1 to LD7, D8 to LD8, D10 to LD9
Changed lines of the file:
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@@
 			)
 		)
-		(property "Value" "SS34 (reverse-polarity)"
-			(at 148.336 29.972 0)
+		(property "Value" "SS34"
+			(at 142.494 29.972 0)
 			(effects
 				(font
@@
 		(on_board yes)
 		(dnp no)
-		(property "Reference" "D8"
+		(property "Reference" "LD8"
 			(at 175.387 242.57 90)
 			(effects
@@
 			(project "WM2-WaterMaster"
 				(path "/00ea9009-1039-4827-8fe4-64ceea0f3b86"
-					(reference "D8")
+					(reference "LD8")
 					(unit 1)
 				)
@@
 		(on_board yes)
 		(dnp no)
-		(property "Reference" "D4"
+		(property "Reference" "LD6"
 			(at 37.338 190.246 90)
 			(effects
@@
 			(project "WM2-WaterMaster"
 				(path "/00ea9009-1039-4827-8fe4-64ceea0f3b86"
-					(reference "D4")
+					(reference "LD6")
 					(unit 1)
 				)
@@
 		(on_board yes)
 		(dnp no)
-		(property "Reference" "D11"
+		(property "Reference" "LD11"
 			(at 177.673 267.335 90)
 			(effects
@@
 			(project "WM2-WaterMaster"
 				(path "/00ea9009-1039-4827-8fe4-64ceea0f3b86"
-					(reference "D11")
+					(reference "LD11")
 					(unit 1)
 				)
@@
 		(on_board yes)
 		(dnp no)
-		(property "Reference" "D5"
+		(property "Reference" "LD4"
 			(at 38.608 84.836 90)
 			(effects
@@
 			(project "WM2-WaterMaster"
 				(path "/00ea9009-1039-4827-8fe4-64ceea0f3b86"
-					(reference "D5")
+					(reference "LD4")
 					(unit 1)
 				)
@@
 		(on_board yes)
 		(dnp no)
-		(property "Reference" "D2"
+		(property "Reference" "LD3"
 			(at 37.338 32.766 90)
 			(effects
@@
 			(project "WPC"
 				(path "/00ea9009-1039-4827-8fe4-64ceea0f3b86"
-					(reference "D2")
+					(reference "LD3")
 					(unit 1)
 				)
@@
 			)
 		)
-		(property "Footprint" "Capacitor_SMD:C_0805_2012Metric"
+		(property "Footprint" "Capacitor_SMD:C_1206_3216Metric_Pad1.33x1.80mm_HandSolder"
 			(at 160.02 39.37 0)
 			(effects
@@
 			)
 		)
-		(property "Footprint" "Capacitor_SMD:C_0805_2012Metric"
+		(property "Footprint" "Capacitor_SMD:C_1206_3216Metric_Pad1.33x1.80mm_HandSolder"
 			(at 209.55 38.1 0)
 			(effects
@@
 		(on_board yes)
 		(dnp no)
-		(property "Reference" "D7"
+		(property "Reference" "LD1"
 			(at 151.003 48.26 90)
 			(effects
@@
 			(project "WM2-WaterMaster"
 				(path "/00ea9009-1039-4827-8fe4-64ceea0f3b86"
-					(reference "D7")
+					(reference "LD1")
 					(unit 1)
 				)
@@
 		(on_board yes)
 		(dnp no)
-		(property "Reference" "D9"
+		(property "Reference" "LD10"
 			(at 175.387 270.51 90)
 			(effects
@@
 			(project "WM2-WaterMaster"
 				(path "/00ea9009-1039-4827-8fe4-64ceea0f3b86"
-					(reference "D9")
+					(reference "LD10")
 					(unit 1)
 				)
@@
 			)
 		)
-		(property "Value" "10mfd,10V tent"
+		(property "Value" "10u/10V tent"
 			(at 353.06 48.006 0)
 			(effects
@@
 			)
 		)
-		(property "Value" "AP63205WU (fixed 5.0V out)"
+		(property "Value" "AP63205WU"
 			(at 185.42 50.038 0)
 			(effects
@@
 			)
 		)
-		(property "Footprint" "Capacitor_SMD:C_0805_2012Metric"
+		(property "Footprint" "Capacitor_SMD:C_1206_3216Metric_Pad1.33x1.80mm_HandSolder"
 			(at 223.52 38.1 0)
 			(effects
@@
 		(on_board yes)
 		(dnp no)
-		(property "Reference" "D12"
+		(property "Reference" "LD2"
 			(at 275.463 104.775 90)
 			(effects
@@
 			(project "WM2-WaterMaster"
 				(path "/00ea9009-1039-4827-8fe4-64ceea0f3b86"
-					(reference "D12")
+					(reference "LD2")
 					(unit 1)
 				)
@@
 		(on_board yes)
 		(dnp no)
-		(property "Reference" "D10"
+		(property "Reference" "LD9"
 			(at 177.673 239.395 90)
 			(effects
@@
 			(project "WM2-WaterMaster"
 				(path "/00ea9009-1039-4827-8fe4-64ceea0f3b86"
-					(reference "D10")
+					(reference "LD9")
 					(unit 1)
 				)
@@
 		(on_board yes)
 		(dnp no)
-		(property "Reference" "D1"
+		(property "Reference" "LD7"
 			(at 36.068 248.666 90)
 			(effects
@@
 			(project "Nursary_OneCH"
 				(path "/00ea9009-1039-4827-8fe4-64ceea0f3b86"
-					(reference "D1")
+					(reference "LD7")
 					(unit 1)
 				)
@@
 		(on_board yes)
 		(dnp no)
-		(property "Reference" "D3"
+		(property "Reference" "LD5"
 			(at 37.338 139.446 90)
 			(effects
@@
 			(project "WM2-WaterMaster"
 				(path "/00ea9009-1039-4827-8fe4-64ceea0f3b86"
-					(reference "D3")
+					(reference "LD5")
 					(unit 1)
 				)
@@
 			)
 		)
-		(property "Value" "10,10V tent"
+		(property "Value" "10u/10V tent"
 			(at 380.492 47.244 0)
 			(effects
