File: products/AWD1-paddy/hardware/AWD-FieldNode/AWD-FieldNode.kicad_sch (KiCad schematic)
At the start: 51 parts, among them J1 SMA 866MHz, J2 PROG, J3 LiFePO4 14500, Q1 AO3401A, Q2 2N7002, SW1 PAIR/BOOT, U1 ESP32-S3-MINI-1-N8, U2 ISC-SX1262-B

Commit message: TH2 field node + common AWD/TH enclosure; AWD v0.2 field charging
TH2 (products/TH-monitor/hardware/TH2-FieldNode):
- Schematic v0.2: ESP32-C3-WROOM-02, SHT40 on the PCB back side,
  LiFePO4 14500 in an on-board AA holder, CN3058E charger (0.31 A),
  RT9080 LDO, 32.768 kHz RTC crystal, magnetic-socket input with USB ESD,
  optional SX1262 LoRa (TH2-W / TH2-L builds). ERC 0 violations.
- Generated from tools/design.py + gen_sch.py (AWD style).
- Enclosure concept v0.3: one 40x60 PCB in the AWD box (shells called
  from awd_enclosure.scad), stacked-plate shield, multi-size pole base,
  and an AWD-vs-TH packaging comparison. Earlier pipe concept archived.
- SMTHSN50-ref: recovered Sasya 2021 Gerbers + schematic (reference only).

AWD (products/AWD1-paddy/hardware/AWD-FieldNode):
- Schematic v0.2: same charging block as TH2 (J4 magnetic socket, F1,
  U5 USBLC6, U3 CN3058E, U4 RT9080, D2/D3, VBUS_DET on IO14); battery
  sense moved to VBAT. ERC 0 violations. PCB not yet updated.
- gen_sch.py keeps the existing root and symbol UUIDs, so the routed
  PCB stays linked (51/51 footprints).
- Project file: restore the RF net class (/RF_ANT 0.36 mm) that a KiCad
  re-save had dropped; add /VBAT, /VBUS, /VBUS_IN to the Power class.
- Enclosure (front/back shell, pipe collar) now tracked.

Co-Authored-By: Claude Opus 5.5 <noreply@anthropic.com>
Parts:
- added C8: 10u, Capacitor_SMD:C_0805_2012Metric, symbol Device:C
- added C9: 1u, Capacitor_SMD:C_0603_1608Metric, symbol Device:C
- added D2: RED, LED_SMD:LED_0603_1608Metric, symbol Device:LED
- added D3: GREEN, LED_SMD:LED_0603_1608Metric, symbol Device:LED
- added F1: 0.5A, Fuse:Fuse_1206_3216Metric, symbol Device:Polyfuse
- added J4: MAG-POGO, Connector_JST:JST_PH_S4B-PH-SM4-TB_1x04-1MP_P2.00mm_Horizontal, symbol Connector_Generic:Conn_01x04
- added R10, R11: 1k, Resistor_SMD:R_0603_1608Metric, symbol Device:R
- added R12, R13: 100k, Resistor_SMD:R_0603_1608Metric, symbol Device:R
- added R8: 0R, Resistor_SMD:R_0603_1608Metric, symbol Device:R
- added R9: 3.9k, Resistor_SMD:R_0603_1608Metric, symbol Device:R
- added U3: CN3058E, Package_SO:SOIC-8-1EP_3.9x4.9mm_P1.27mm_EP2.41x3.3mm_ThermalVias, symbol AWD:CN3058E
- added U4: RT9080-33GJ5, Package_TO_SOT_SMD:SOT-23-5, symbol Regulator_Linear:AP2112K-3.3
- added U5: USBLC6-2SC6, Package_TO_SOT_SMD:SOT-23-6, symbol Power_Protection:USBLC6-2SC6
- TP1: value T14 -> VBUS_DET
Connections:
- net +3V3: now also U4.5 (VOUT); no longer C1.1, Q1.2 (S), R4.1
- net GND: now also C8.2, C9.2, J4.4 (Pin_4), R13.2, R8.2, R9.2, U3.3 (GND), U3.9 (EP), U4.2 (GND), U5.2 (GND)
- net USB_DN: now also J4.2 (Pin_2), U5.1 (I/O1), U5.6 (I/O1)
- net USB_DP: now also J4.3 (Pin_3), U5.3 (I/O2), U5.4 (I/O2)
- net T14_SPARE renamed VBUS_DET
- net VBUS_DET: now also R12.2, R13.1
- new net CHG_A: D2.2 (A), R10.2
- new net CHG_ISET: R9.1, U3.2 (ISET)
- new net CHG_TEMP: R8.1, U3.1 (TEMP)
- new net CHRG_N: D2.1 (K), U3.7 (~{CHRG})
- new net DONE_A: D3.2 (A), R11.2
- new net DONE_N: D3.1 (K), U3.6 (~{DONE})
- new net VBAT: C1.1, C9.1, Q1.2 (S), R4.1, U3.5 (BAT), U4.1 (VIN), U4.3 (EN)
- new net VBUS: C8.1, F1.2, R10.1, R11.1, R12.1, U3.4 (VIN), U3.8 (CE), U5.5 (VBUS)
- new net VBUS_IN: F1.1, J4.1 (Pin_1)
Other:
- note added: "Battery sense: Q2 enables the 1M/1M divider (from VBAT) only while sampling VBAT_ADC (ADC2, WiFi off)."
- note added: "Power: LiFePO4 14500 -> Q1 reverse protection -> VBAT -> U4 RT9080 LDO (2 uA Iq) -> +3V3. VBAT reaches 3.6 V while charging."
- note added: "U5 = USB ESD. RED = charging, GREEN = full. VBUS_DET on IO14 wakes the S3."
- note added: "v0.2 field charging: J4 magnetic socket -> F1 -> U3 CN3058E (0.31 A, 3.6 V)."
- note removed: "Battery sense: Q2 enables the 1M/1M divider only while sampling VBAT_ADC (ADC2, WiFi off)."
- note removed: "Power: LiFePO4 14500 straight onto the 3V3 rail (3.0-3.4 V plateau, no regulator, ~0 uA quiescent). Q1 = reverse-polarity protection."
